Commit message: Taller gates to match IRL ones

File: safe_control_gym/envs/gym_pybullet_drones/assets/portal.urdf (robot description, URDF)
Before this commit: robot architrave, 6 links, 5 joints
Links:
- link support: geometry collision cylinder length=.8 radius=0.05; visual cylinder length=.8 radius=0.05
