Commit message: Logging

File: safe_control_gym/envs/gym_pybullet_drones/assets/obstacle.urdf (robot description, URDF)
Before this commit: robot architrave, 1 links, 0 joints
Links:
- link base_link: geometry collision cylinder length=.8 radius=0.1; visual cylinder length=.8 radius=0.1

File: safe_control_gym/envs/gym_pybullet_drones/assets/portal.urdf (robot description, URDF)
Before this commit: robot architrave, 1 links, 0 joints
Links:
- added link blue_edge, mass 0.3; collision box size=.4 .05 .05; visual box size=.4 .05 .05
- added link green_edge, mass 0.3; collision box size=.4 .05 .05; visual box size=.4 .05 .05
- added link grey_edge, mass 0.3; collision box size=.4 .05 .05; visual box size=.4 .05 .05
- added link red_edge, mass 0.3; collision box size=.4 .05 .05; visual box size=.4 .05 .05
- link base_link: mass 0.3 -> None; geometry visual sphere radius=0.03
Joints:
- added joint blue_joint: type fixed, parent base_link, child blue_edge
- added joint green_joint: type fixed, parent base_link, child green_edge
- added joint grey_joint: type fixed, parent base_link, child grey_edge
- added joint red_joint: type fixed, parent base_link, child red_edge

Commit message: Simple map

File: safe_control_gym/envs/gym_pybullet_drones/assets/obstacle.urdf (robot description, URDF)
Before this commit: robot architrave, 1 links, 0 joints
Links:
- link base_link: mass 0.3 -> 2.0; geometry collision cylinder length=1.5 radius=0.075; visual cylinder length=1.5 radius=0.075

File: safe_control_gym/envs/gym_pybullet_drones/assets/portal.urdf (robot description, URDF)
Before this commit: robot architrave, 5 links, 4 joints
Links:
- added link support, mass 1.0; collision cylinder length=1.0 radius=0.05; visual cylinder length=1.0 radius=0.05
- link base_link: geometry visual sphere radius=0.01
- link blue_edge: mass 0.3 -> 0.25; geometry collision box size=.5 .05 .05; visual box size=.5 .05 .05
- link green_edge: mass 0.3 -> 0.25; geometry collision box size=.5 .05 .05; visual box size=.5 .05 .05
- link grey_edge: mass 0.3 -> 0.25; geometry collision box size=.5 .05 .05; visual box size=.5 .05 .05
- link red_edge: mass 0.3 -> 0.25; geometry collision box size=.5 .05 .05; visual box size=.5 .05 .05
Joints:
- added joint support_joint: type fixed, parent base_link, child support

Commit message: Real obstacles height

File: safe_control_gym/envs/gym_pybullet_drones/assets/obstacle.urdf (robot description, URDF)
Before this commit: robot architrave, 1 links, 0 joints
Links:
- link base_link: geometry collision cylinder length=0.8 radius=0.05; visual cylinder length=0.8 radius=0.05

File: safe_control_gym/envs/gym_pybullet_drones/assets/portal.urdf (robot description, URDF)
Before this commit: robot architrave, 6 links, 5 joints
Links:
- link support: geometry collision cylinder length=.5 radius=0.05; visual cylinder length=.5 radius=0.05

Commit message: Taller obstacles

File: safe_control_gym/envs/gym_pybullet_drones/assets/obstacle.urdf (robot description, URDF)
Before this commit: robot architrave, 1 links, 0 joints
Links:
- added link box_link, mass 0.25; collision box size=.15 .15 .25; visual box size=.15 .15 .25
Joints:
- added joint box_joint: type fixed, parent base_link, child box_link

Commit message: increase the heights of the obstacles to 1.3 m

File: safe_control_gym/envs/gym_pybullet_drones/assets/obstacle.urdf (robot description, URDF)
Before this commit: robot architrave, 2 links, 1 joints
Links:
- link base_link: geometry collision cylinder length=1.05 radius=0.05; visual cylinder length=1.05 radius=0.05
