Commit message: Finish primary refactor. Add tests.

File: safe_control_gym/envs/assets/gate.urdf (robot description, URDF)
Before this commit: robot gate, 1 links, 0 joints
Links:
- added link blue_edge, mass 0.0; collision box size=.5 .05 .05; visual box size=.5 .05 .05
- added link green_edge, mass 0.0; collision box size=.5 .05 .05; visual box size=.5 .05 .05
- added link grey_edge, mass 0.0; collision box size=.5 .05 .05; visual box size=.5 .05 .05
- added link red_edge, mass 0.0; collision box size=.5 .05 .05; visual box size=.5 .05 .05
- added link support, mass 0.0; collision cylinder length=.8 radius=0.05; visual cylinder length=.8 radius=0.05
- link base_link: mass 0. -> 0.0; geometry visual sphere radius=0.01
Joints:
- added joint blue_joint: type fixed, parent base_link, child blue_edge
- added joint green_joint: type fixed, parent base_link, child green_edge
- added joint grey_joint: type fixed, parent base_link, child grey_edge
- added joint red_joint: type fixed, parent base_link, child red_edge
- added joint support_joint: type fixed, parent base_link, child support, origin xyz=0 0 -0.6 rpy=0 0 0

File: safe_control_gym/envs/assets/obstacle.urdf (robot description, URDF)
Before this commit: robot architrave, 2 links, 1 joints
Links:
- added link cylinder_link, mass 2.0; collision cylinder length=0.8 radius=0.05; visual cylinder length=0.8 radius=0.05
- link base_link: mass 2.0 -> 0.01; geometry visual sphere radius=.01
Joints:
- added joint cylinder_joint: type fixed, parent base_link, child cylinder_link, origin xyz=0.0 0.0 -0.4 rpy=0 0 0
- joint box_joint: origin (none) -> xyz=0.0 0.0 -0.525 rpy=0 0 0; parent base_link -> cylinder_link
